File: RasPi-BplusHAT.brd (EAGLE design)
At the start: 65 x 56 mm, 14 parts, among them K1 PIN20X2, U1 EEPROM24

Commit message: Add files via upload
Routing:
- net N$2: track 26.3 -> 27.2 mm
Changed lines of the file:
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@@
 <wire x1="56.9976" y1="32.512" x2="56.945" y2="32.4975" width="0.254" layer="1"/>
 <wire x1="60.0456" y1="32.512" x2="60.075" y2="32.4975" width="0.254" layer="1"/>
-<wire x1="54.6608" y1="35.3568" x2="55.1688" y2="35.3568" width="0.254" layer="1"/>
-<wire x1="53.7464" y1="36.2712" x2="54.6608" y2="35.3568" width="0.254" layer="1"/>
-<wire x1="53.7464" y1="36.9824" x2="53.7464" y2="36.2712" width="0.254" layer="1"/>
+<wire x1="54.0258" y1="35.3568" x2="55.1688" y2="35.3568" width="0.254" layer="1"/>
+<wire x1="53.7464" y1="35.6362" x2="54.0258" y2="35.3568" width="0.254" layer="1"/>
+<wire x1="53.7464" y1="36.9824" x2="53.7464" y2="35.6362" width="0.254" layer="1"/>
 <wire x1="54.0512" y1="37.2872" x2="53.7464" y2="36.9824" width="0.254" layer="1"/>
-<wire x1="56.388" y1="37.2872" x2="54.0512" y2="37.2872" width="0.254" layer="1"/>
-<wire x1="56.9976" y1="36.6776" x2="56.8452" y2="36.83" width="0.254" layer="1"/>
-<wire x1="56.8452" y1="36.83" x2="56.388" y2="37.2872" width="0.254" layer="1"/>
-<wire x1="56.9976" y1="32.6136" x2="56.9976" y2="36.6776" width="0.254" layer="1"/>
+<wire x1="56.4515" y1="37.2872" x2="54.0512" y2="37.2872" width="0.254" layer="1"/>
+<wire x1="56.9976" y1="36.7919" x2="57.0357" y2="36.83" width="0.254" layer="1"/>
+<wire x1="56.9722" y1="36.7665" x2="56.4515" y2="37.2872" width="0.254" layer="1"/>
+<wire x1="56.9976" y1="32.6136" x2="56.9976" y2="36.7919" width="0.254" layer="1"/>
 <wire x1="55.1688" y1="35.3568" x2="55.205" y2="35.355" width="0.254" layer="1"/>
 <wire x1="56.9976" y1="32.6136" x2="56.945" y2="32.4975" width="0.254" layer="1"/>
-<wire x1="56.8452" y1="36.83" x2="61.976" y2="41.9608" width="0.254" layer="1"/>
-<wire x1="61.976" y1="41.9608" x2="62.025" y2="42.0225" width="0.254" layer="1"/>
+<wire x1="56.9722" y1="36.7665" x2="56.9976" y2="36.7919" width="0.254" layer="1"/>
+<wire x1="57.0357" y1="36.83" x2="61.241" y2="41.0353" width="0.254" layer="1"/>
+<wire x1="61.241" y1="41.0353" x2="62.025" y2="42.0225" width="0.254" layer="1"/>
 <wire x1="42.9768" y1="36.9824" x2="53.7464" y2="36.9824" width="0.254" layer="1"/>
 <wire x1="28.7528" y1="51.2064" x2="42.9768" y2="36.9824" width="0.254" layer="1"/>
@@
 <contactref element="R1" pad="1"/>
 <contactref element="K1" pad="28"/>
-<wire x1="59.8424" y1="41.9608" x2="60.0456" y2="41.9608" width="0.254" layer="1"/>
-<wire x1="55.7784" y1="37.8968" x2="59.8424" y2="41.9608" width="0.254" layer="1"/>
-<wire x1="55.2704" y1="37.8968" x2="55.7784" y2="37.8968" width="0.254" layer="1"/>
-<wire x1="60.0456" y1="41.9608" x2="60.125" y2="42.0225" width="0.254" layer="1"/>
+<wire x1="60.125" y1="42.0225" x2="60.125" y2="41.7354" width="0.254" layer="1"/>
+<wire x1="60.125" y1="41.7354" x2="56.2864" y2="37.8968" width="0.254" layer="1"/>
+<wire x1="55.2704" y1="37.8968" x2="56.2864" y2="37.8968" width="0.254" layer="1"/>
 <wire x1="55.2704" y1="37.8968" x2="55.205" y2="37.895" width="0.254" layer="1"/>
 <wire x1="41.3512" y1="52.7304" x2="41.3512" y2="53.7464" width="0.254" layer="1"/>
@@
 <contactref element="R2" pad="1"/>
 <contactref element="K1" pad="27"/>
-<wire x1="60.0456" y1="43.9928" x2="60.0456" y2="44.5008" width="0.254" layer="1"/>
-<wire x1="55.2704" y1="39.2176" x2="60.0456" y2="43.9928" width="0.254" layer="1"/>
 <wire x1="60.0456" y1="44.5008" x2="60.125" y2="44.5625" width="0.254" layer="1"/>
-<wire x1="55.2704" y1="39.2176" x2="55.205" y2="39.165" width="0.254" layer="1"/>
+<wire x1="55.3194" y1="39.165" x2="55.205" y2="39.165" width="0.254" layer="1"/>
 <wire x1="42.4688" y1="51.2064" x2="41.4528" y2="51.2064" width="0.254" layer="1"/>
 <wire x1="54.4576" y1="39.2176" x2="42.4688" y2="51.2064" width="0.254" layer="1"/>
@@
 <wire x1="41.4528" y1="51.2064" x2="41.39" y2="51.23" width="0.254" layer="1"/>
 <wire x1="55.1688" y1="39.2176" x2="55.205" y2="39.165" width="0.254" layer="1"/>
+<wire x1="55.205" y1="39.165" x2="56.6275" y2="39.165" width="0.254" layer="1"/>
+<wire x1="56.6275" y1="39.165" x2="58.293" y2="40.8305" width="0.254" layer="1"/>
+<wire x1="58.293" y1="40.8305" x2="58.293" y2="42.7482" width="0.254" layer="1"/>
+<wire x1="58.293" y1="42.7482" x2="60.0456" y2="44.5008" width="0.254" layer="1"/>
 </signal>
 <signal name="N$3">
