File: RasPi-BplusHAT-3v3.brd (EAGLE design)
At the start: 65 x 56 mm, 14 parts, among them K1 PIN20X2, U1 EEPROM24

Commit message: Add files via upload
Parts:
- removed R5, R6: 3K3, SparkFun-Resistors:AXIAL-0.3
- moved R7 5.24 mm to (19.7, 38.7), turned to 90 degrees
- moved R4 3.59 mm to (15.9, 38.7), turned to 90 degrees
Connections:
- net GND: no longer R5.P$1, R6.P$1
- net MAIX-UART0-RX: now also R4.P$1; no longer R4.P$2
- net MAIX-UART0-TX: now also R7.P$1; no longer R7.P$2
- net RPI-UART-RX: now also R7.P$2; no longer R6.P$2, R7.P$1
- net RPI-UART-TX: now also R4.P$2; no longer R4.P$1, R5.P$2
Routing:
- net RPI-UART-RX: track 37.3 -> 11.7 mm
- net MAIX-UART0-RX: track 43.5 -> 34.3 mm
- net RPI-UART-TX: track 20.2 -> 12.2 mm
- net MAIX-UART0-TX: track 33.8 -> 40.2 mm
Changed lines of the file:
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@@
 </element>
 <element name="FRAME1" library="SparkFun-Aesthetics" library_urn="urn:adsk.eagle:library:507" package="CREATIVE_COMMONS" package3d_urn="urn:adsk.eagle:package:37121/1" value="FRAME-LETTER" x="3.22" y="-9.84" smashed="yes"/>
-<element name="R5" library="SparkFun-Resistors" library_urn="urn:adsk.eagle:library:532" package="AXIAL-0.3" package3d_urn="urn:adsk.eagle:package:39658/1" value="3K3" x="31.115" y="41.275" smashed="yes" rot="R180">
-<attribute name="NAME" x="31.115" y="40.259" size="0.6096" layer="25" font="vector" ratio="20" rot="R180" align="bottom-center"/>
-<attribute name="PROD_ID" value=" " x="31.115" y="41.275" size="1.778" layer="27" rot="R180" display="off"/>
-<attribute name="VALUE" x="31.115" y="42.291" size="0.6096" layer="27" font="vector" ratio="20" rot="R180" align="top-center"/>
+<element name="R4" library="SparkFun-Resistors" library_urn="urn:adsk.eagle:library:532" package="AXIAL-0.3" package3d_urn="urn:adsk.eagle:package:39658/1" value="2K2" x="15.875" y="38.735" smashed="yes" rot="R90">
+<attribute name="NAME" x="14.859" y="38.735" size="0.6096" layer="25" font="vector" ratio="20" rot="R90" align="bottom-center"/>
+<attribute name="PROD_ID" value=" " x="15.875" y="38.735" size="1.778" layer="27" rot="R90" display="off"/>
+<attribute name="VALUE" x="16.891" y="38.735" size="0.6096" layer="27" font="vector" ratio="20" rot="R90" align="top-center"/>
 </element>
-<element name="R4" library="SparkFun-Resistors" library_urn="urn:adsk.eagle:library:532" package="AXIAL-0.3" package3d_urn="urn:adsk.eagle:package:39658/1" value="2K2" x="18.415" y="41.275" smashed="yes" rot="R180">
-<attribute name="NAME" x="18.415" y="40.259" size="0.6096" layer="25" font="vector" ratio="20" rot="R180" align="bottom-center"/>
-<attribute name="PROD_ID" value=" " x="18.415" y="41.275" size="1.778" layer="27" rot="R180" display="off"/>
-<attribute name="VALUE" x="18.415" y="42.291" size="0.6096" layer="27" font="vector" ratio="20" rot="R180" align="top-center"/>
-</element>
-<element name="R6" library="SparkFun-Resistors" library_urn="urn:adsk.eagle:library:532" package="AXIAL-0.3" package3d_urn="urn:adsk.eagle:package:39658/1" value="3K3" x="31.115" y="33.655" smashed="yes" rot="R180">
-<attribute name="NAME" x="31.115" y="32.639" size="0.6096" layer="25" font="vector" ratio="20" rot="R180" align="bottom-center"/>
-<attribute name="PROD_ID" value=" " x="31.115" y="33.655" size="1.778" layer="27" rot="R180" display="off"/>
-<attribute name="VALUE" x="31.115" y="34.671" size="0.6096" layer="27" font="vector" ratio="20" rot="R180" align="top-center"/>
-</element>
-<element name="R7" library="SparkFun-Resistors" library_urn="urn:adsk.eagle:library:532" package="AXIAL-0.3" package3d_urn="urn:adsk.eagle:package:39658/1" value="2K2" x="18.415" y="33.655" smashed="yes" rot="R180">
-<attribute name="NAME" x="18.415" y="32.639" size="0.6096" layer="25" font="vector" ratio="20" rot="R180" align="bottom-center"/>
-<attribute name="PROD_ID" value=" " x="19.415" y="33.655" size="1.778" layer="27" rot="R180" display="off"/>
-<attribute name="VALUE" x="18.415" y="34.671" size="0.6096" layer="27" font="vector" ratio="20" rot="R180" align="top-center"/>
+<element name="R7" library="SparkFun-Resistors" library_urn="urn:adsk.eagle:library:532" package="AXIAL-0.3" package3d_urn="urn:adsk.eagle:package:39658/1" value="2K2" x="19.685" y="38.735" smashed="yes" rot="R90">
+<attribute name="NAME" x="18.669" y="38.735" size="0.6096" layer="25" font="vector" ratio="20" rot="R90" align="bottom-center"/>
+<attribute name="PROD_ID" value=" " x="19.685" y="37.735" size="1.778" layer="27" rot="R90" display="off"/>
+<attribute name="VALUE" x="20.701" y="38.735" size="0.6096" layer="27" font="vector" ratio="20" rot="R90" align="top-center"/>
 </element>
 </elements>
@@
 </polygon>
 <contactref element="P4" pad="1"/>
-<contactref element="R5" pad="P$1"/>
-<contactref element="R6" pad="P$1"/>
 </signal>
 <signal name="+3V3">
@@
 <contactref element="P4" pad="2"/>
 <wire x1="10.91" y1="53.77" x2="12.192" y2="52.488" width="0.6096" layer="1" curve="-90"/>
-<wire x1="12.192" y1="46.99" x2="14.732" y2="44.45" width="0.6096" layer="1" curve="90"/>
-<wire x1="15.875" y1="44.45" x2="18.415" y2="41.91" width="0.6096" layer="1" curve="-90"/>
-<wire x1="18.415" y1="26.035" x2="20.955" y2="23.495" width="0.6096" layer="1" curve="90"/>
-<wire x1="20.955" y1="23.495" x2="38.735" y2="23.495" width="0.6096" layer="1"/>
-<wire x1="12.192" y1="52.488" x2="12.192" y2="46.99" width="0.6096" layer="1"/>
-<wire x1="14.732" y1="44.45" x2="15.875" y2="44.45" width="0.6096" layer="1"/>
-<wire x1="18.415" y1="41.91" x2="18.415" y2="26.035" width="0.6096" layer="1"/>
 <wire x1="10.91" y1="53.77" x2="8.37" y2="53.77" width="0.6096" layer="1"/>
+<wire x1="12.192" y1="39.878" x2="14.732" y2="37.338" width="0.6096" layer="1" curve="90"/>
+<wire x1="27.94" y1="37.338" x2="30.48" y2="34.798" width="0.6096" layer="1" curve="-90"/>
+<wire x1="30.48" y1="26.035" x2="33.02" y2="23.495" width="0.6096" layer="1" curve="90"/>
+<wire x1="33.02" y1="23.495" x2="38.735" y2="23.495" width="0.6096" layer="1"/>
+<wire x1="12.192" y1="52.488" x2="12.192" y2="39.878" width="0.6096" layer="1"/>
+<wire x1="14.732" y1="37.338" x2="27.94" y2="37.338" width="0.6096" layer="1"/>
+<wire x1="30.48" y1="34.798" x2="30.48" y2="26.035" width="0.6096" layer="1"/>
 </signal>
 <signal name="PF6">
@@
 <signal name="MAIX-UART0-TX">
 <contactref element="P5" pad="10"/>
-<contactref element="R7" pad="P$2"/>
-<wire x1="14.605" y1="33.655" x2="14.605" y2="5.715" width="0.254" layer="1"/>
-<wire x1="14.605" y1="5.715" x2="12.065" y2="3.175" width="0.254" layer="1" curve="-90"/>
-<wire x1="12.065" y1="3.175" x2="9.749790625" y2="3.175" width="0.254" layer="1"/>
+<contactref element="R7" pad="P$1"/>
+<wire x1="19.685" y1="34.925" x2="19.685" y2="5.715" width="0.254" layer="1"/>
+<wire x1="19.685" y1="5.715" x2="17.145" y2="3.175" width="0.254" layer="1" curve="-90"/>
+<wire x1="17.145" y1="3.175" x2="9.749790625" y2="3.175" width="0.254" layer="1"/>
 </signal>
 <signal name="MAIX-UART0-RX">
 <contactref element="P5" pad="9"/>
-<contactref element="R4" pad="P$2"/>
-<wire x1="14.605" y1="41.275" x2="9.271" y2="41.275" width="0.254" layer="1"/>
-<wire x1="9.271" y1="41.275" x2="6.731" y2="38.735" width="0.254" layer="1" curve="90"/>
-<wire x1="6.731" y1="8.255" x2="9.271" y2="5.715" width="0.254" layer="1" curve="90"/>
 <wire x1="9.271" y1="5.715" x2="9.749790625" y2="5.715" width="0.254" layer="1"/>
-<wire x1="6.731" y1="38.735" x2="6.731" y2="8.255" width="0.254" layer="1"/>
+<contactref element="R4" pad="P$1"/>
+<wire x1="15.875" y1="34.925" x2="15.875" y2="8.255" width="0.254" layer="1"/>
+<wire x1="15.875" y1="8.255" x2="13.335" y2="5.715" width="0.254" layer="1" curve="-90"/>
+<wire x1="13.335" y1="5.715" x2="9.749790625" y2="5.715" width="0.254" layer="1"/>
 </signal>
 <signal name="PH6">
@@
 </signal>
 <signal name="RPI-UART-RX">
-<contactref element="R6" pad="P$2"/>
-<contactref element="R7" pad="P$1"/>
 <contactref element="K1" pad="10"/>
-<wire x1="22.225" y1="33.655" x2="27.305" y2="33.655" width="0.254" layer="1"/>
-<wire x1="18.53" y1="53.77" x2="19.8755" y2="52.4245" width="0.254" layer="1" curve="-90"/>
-<wire x1="19.8755" y1="52.4245" x2="19.8755" y2="49.3395" width="0.254" layer="1"/>
-<wire x1="19.8755" y1="49.3395" x2="20.955" y2="48.26" width="0.254" layer="1" curve="90"/>
-<wire x1="28.6385" y1="48.26" x2="31.1785" y2="45.72" width="0.254" layer="1" curve="-90"/>
-<wire x1="31.1785" y1="36.195" x2="28.6385" y2="33.655" width="0.254" layer="1" curve="-90"/>
-<wire x1="28.6385" y1="33.655" x2="27.305" y2="33.655" width="0.254" layer="1"/>
-<wire x1="20.955" y1="48.26" x2="28.6385" y2="48.26" width="0.254" layer="1"/>
-<wire x1="31.1785" y1="45.72" x2="31.1785" y2="36.195" width="0.254" layer="1"/>
+<contactref element="R7" pad="P$2"/>
+<wire x1="18.53" y1="53.77" x2="19.685" y2="52.615" width="0.254" layer="1" curve="-90"/>
+<wire x1="19.685" y1="52.615" x2="19.685" y2="42.545" width="0.254" layer="1"/>
 </signal>
 <signal name="RPI-UART-TX">
-<contactref element="R5" pad="P$2"/>
-<contactref element="R4" pad="P$1"/>
 <contactref element="K1" pad="8"/>
-<wire x1="27.305" y1="41.275" x2="22.225" y2="41.275" width="0.254" layer="1"/>
-<wire x1="22.225" y1="41.275" x2="20.32" y2="43.18" width="0.254" layer="1" curve="-90"/>
-<wire x1="20.32" y1="43.18" x2="20.32" y2="45.72" width="0.254" layer="1"/>
-<wire x1="20.32" y1="45.72" x2="19.05" y2="46.99" width="0.254" layer="1" curve="90"/>
-<wire x1="19.05" y1="46.99" x2="17.272" y2="48.768" width="0.254" layer="1" curve="-90"/>
-<wire x1="17.272" y1="52.488" x2="15.99" y2="53.77" width="0.254" layer="1" curve="90"/>
-<wire x1="17.272" y1="48.768" x2="17.272" y2="52.488" width="0.254" layer="1"/>
+<contactref element="R4" pad="P$2"/>
+<wire x1="15.875" y1="42.545" x2="15.875" y2="45.085" width="0.254" layer="1"/>
+<wire x1="15.875" y1="45.085" x2="16.51" y2="45.72" width="0.254" layer="1" curve="-90"/>
+<wire x1="16.51" y1="45.72" x2="17.145" y2="46.355" width="0.254" layer="1" curve="90"/>
+<wire x1="17.145" y1="52.615" x2="15.99" y2="53.77" width="0.254" layer="1" curve="90"/>
+<wire x1="17.145" y1="46.355" x2="17.145" y2="52.615" width="0.254" layer="1"/>
 </signal>
 </signals>
